File: Delta_DPS-1125AB_1450W/Schematics/DC_DC.kicad_sch (KiCad schematic)
At the start: 29 parts, among them Q1 Q_NMOS, Q10 Q_NMOS, Q2 Q_NMOS, Q3 Q_NMOS, Q4 Q_NMOS, Q5 Q_NMOS, Q6 Q_NMOS, Q7 Q_NMOS, Q8 Q_NMOS, Q9 Q_NMOS, T1 prim: 23 turns

Commit message: pdf generation
Parts:
- added C15: 470µF 36v, symbol Device:C_Polarized
- added C16: 100µF 16v, symbol Device:C_Polarized
- added C17: C, symbol Device:C
- added D3: D, symbol Device:D
- added D7: D_Zener, symbol Device:D_Zener
- added R21: 10K, symbol Device:R_US
- added R22: 200, symbol Device:R_US
- added R23: 0.22R 1/2W, symbol Device:R_US
- added U2: L7912, symbol Regulator_Linear:L7912
Connections:
- net GND: now also C15.1, C16.1, C17.1, D3.1 (K), R21.2, R22.2, U2.1 (GND)
- net aux2: now reaches L1.1
- net aux2: now also C15.2, U2.2 (VI)
- net aux1: now reaches L1.2
- net aux1: now also D3.2 (A), R23.1
- new net: D7.1 (K), R22.1
- new net: C17.2, R23.2
- new net 12VN: C16.2, D7.2 (A), R21.1, U2.3 (VO)
Other:
- note added: "Auxilary -12V"
- note added: "Secondary winding 10 turns Coupled inductor (Auxiliary -12V circuit)"
- note removed: "Secondary winding 10 turns For current sensing"
- moved on the sheet: C1, C2, C3, C5, C6, C8, Q1, Q10, Q2, Q3, Q4, Q5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
