File: Delta_DPS-1125AB_1450W/Schematics/EMI_FILTER.kicad_sch (KiCad schematic)
At the start: 23 parts

Commit message: pdf generation
Parts:
- added CY7: 0.33µF, symbol Device:C_Small
- added CY8, CY9: 470pF, symbol Device:C_Small
Connections:
- net Earth: now also CY8.2, CY9.2
- net L: now also CY7.1, CY8.1
- net N: now also CY7.2, CY9.1
Other:
- note added: "0.33µF K MKP-X2 310V-250v~ 40/110/56/B"
- note added: "AC371k x1: 400v y2: 250v"
- note added: "Inline EMI filter"
- note added: "Wire common choke core 2 turns"
- note removed: "Wire common choke core"
